File: PCB/final_project/final_project_v0.1/final_project_v0.1.kicad_sch (KiCad schematic)
At the start: 4 parts, among them J1 USB_C_Receptacle_USB2.0_16P, U1 ESP32-S3-WROOM-1, U2 TC1262-33

Commit message: Notebook Update
Parts:
- added AudioAmplifier1: MAX98357A, Connector_PinHeader_2.54mm:PinHeader_1x07_P2.54mm_Vertical, symbol Connector:Conn_01x07_Pin
- added C2, C4: 0.1u, Capacitor_SMD:C_0805_2012Metric_Pad1.18x1.45mm_HandSolder, symbol Device:C
- added C3, C6: 10u, Capacitor_SMD:C_0805_2012Metric_Pad1.18x1.45mm_HandSolder, symbol Device:C
- added C5, C7, C8: 1u, Capacitor_SMD:C_0805_2012Metric_Pad1.18x1.45mm_HandSolder, symbol Device:C
- added DebugSerialPort1: Conn_01x06_Pin, Connector_PinHeader_2.54mm:PinHeader_1x06_P2.54mm_Vertical, symbol Connector:Conn_01x06_Pin
- added J10, J11, J5, J6, J7, J8, J9: Conn_01x02_Pin, Connector_PinHeader_2.54mm:PinHeader_1x02_P2.54mm_Vertical, symbol Connector:Conn_01x02_Pin
- added J2, LCDDisplay1: Conn_01x04_Pin, Connector_PinHeader_2.54mm:PinHeader_1x04_P2.54mm_Vertical, symbol Connector:Conn_01x04_Pin
- added J3, J4: Conn_01x03_Pin, Connector_PinHeader_2.54mm:PinHeader_1x03_P2.54mm_Vertical, symbol Connector:Conn_01x03_Pin
- added MICCLK1, MICDA1: Conn_01x03_Socket, Connector_PinHeader_2.54mm:PinHeader_1x03_P2.54mm_Vertical, symbol Connector:Conn_01x03_Socket
- added Q1, Q2: SS8050-G, Custom:TRAN_SS8050-G_CIP, symbol Custom:SS8050-G
- added R1, R6, R7: 100k, Resistor_SMD:R_0805_2012Metric_Pad1.20x1.40mm_HandSolder, symbol Device:R
- added R10, R11, R2, R3, R8, R9: 10k, Resistor_SMD:R_0805_2012Metric_Pad1.20x1.40mm_HandSolder, symbol Device:R
- added R4, R5: 4.7k, Resistor_SMD:R_0805_2012Metric_Pad1.20x1.40mm_HandSolder, symbol Device:R
- added SW1, SW2, SW3: SW_Push, Button_Switch_THT:SW_PUSH_6mm_H4.3mm, symbol Switch:SW_Push
- C1: footprint (none) -> Capacitor_SMD:C_0805_2012Metric_Pad1.18x1.45mm_HandSolder
- J1: footprint (none) -> Connector_USB:USB_C_Receptacle_GCT_USB4085
- U2: footprint (none) -> Package_TO_SOT_SMD:SOT-223-3_TabPin2
Connections:
- net +3V3: now also U1.2 (3V3), AudioAmplifier1.7 (Pin_7), C2.1, C3.1, C4.1, MICCLK1.1 (Pin_1), R3.1, R6.1, R7.1, SW1.1
- net +5V: now also C6.1, LCDDisplay1.2 (Pin_2), R4.1, R5.1
- net GND: now also U1.1 (GND), U1.40 (GND), U1.41 (GND), AudioAmplifier1.6 (Pin_6), C2.2, C3.2, C4.2, C5.2, C6.2, C7.2, C8.2, DebugSerialPort1.1 (Pin_1), LCDDisplay1.1 (Pin_1), MICDA1.3 (Pin_3), R1.1, R2.1, SW2.2, SW3.2
- net 17: now reaches U1.10 (IO17)
- net 17: now also J3.3 (Pin_3)
- net MICSDA: now reaches U1.11 (IO18)
- net MICSDA: now also MICDA1.2 (Pin_2), R1.2
- net MICEN: now reaches U1.12 (IO8)
- net MICEN: now also MICDA1.1 (Pin_1), R2.2, SW1.2
- net 19: now reaches U1.13 (IO19)
- net 19: now also J5.1 (Pin_1)
- net 20: now reaches U1.14 (IO20)
- net 20: now also J5.2 (Pin_2)
- net IO3: now reaches U1.15 (IO3)
- net IO3: now also J10.1 (Pin_1)
- net 46: now reaches U1.16 (IO46)
- net 46: now also J10.2 (Pin_2)
- net 9: now reaches U1.17 (IO9)
- net 9: now also J4.1 (Pin_1)
- net 10: now reaches U1.18 (IO10)
- net 10: now also J4.2 (Pin_2)
- net 11: now reaches U1.19 (IO11)
- net 11: now also J4.3 (Pin_3)
- net A_LRCLK: now reaches U1.20 (IO12)
- net A_LRCLK: now also AudioAmplifier1.1 (Pin_1)
- net A_BCLK: now reaches U1.21 (IO13)
- net A_BCLK: now also AudioAmplifier1.2 (Pin_2)
- net A_Din: now reaches U1.22 (IO14)
- net A_Din: now also AudioAmplifier1.3 (Pin_3)
- net A_GAIN: now reaches U1.23 (IO21)
- net A_GAIN: now also AudioAmplifier1.4 (Pin_4)
- net A_SDMODEB: now reaches U1.24 (IO47)
- net A_SDMODEB: now also AudioAmplifier1.5 (Pin_5)
- net 48: now reaches U1.25 (IO48)
- net 48: now also J7.2 (Pin_2)
- net 45: now reaches U1.26 (IO45)
- net 45: now also J7.1 (Pin_1)
- net GPIO_Strapping: now reaches U1.27 (IO0)
- net GPIO_Strapping: now also C8.1, R7.2, R9.2, SW3.1
- net 35: now reaches U1.28 (IO35)
- net 35: now also J2.1 (Pin_1)
- net 36: now reaches U1.29 (IO36)
- net 36: now also J2.2 (Pin_2)
- net Chip_EN: now reaches U1.3 (EN)
- net Chip_EN: now also C7.1, R6.2, R8.2, SW2.1
- net 37: now reaches U1.30 (IO37)
- net 37: now also J2.3 (Pin_3)
- net 38: now reaches U1.31 (IO38)
- net 38: now also J2.4 (Pin_4)
- net SDA_LCD: now reaches U1.32 (IO39)
- net SDA_LCD: now also LCDDisplay1.3 (Pin_3), R5.2
- net SCL_LCD: now reaches U1.33 (IO40)
- net SCL_LCD: now also LCDDisplay1.4 (Pin_4), R4.2
- net 41: now reaches U1.34 (IO41)
- net 41: now also J9.1 (Pin_1)
- net 42: now reaches U1.35 (IO42)
- net 42: now also J9.2 (Pin_2)
- net TXS: now reaches U1.36 (RXD0)
- net TXS: now also DebugSerialPort1.4 (Pin_4)
- net RXS: now reaches U1.37 (TXD0)
- net RXS: now also DebugSerialPort1.5 (Pin_5)
- net 2: now reaches U1.38 (IO2)
- net 2: now also J6.2 (Pin_2)
- net 1: now reaches U1.39 (IO1)
- net 1: now also J6.1 (Pin_1)
- net MICSCK: now reaches U1.4 (IO4)
- net MICSCK: now also MICCLK1.2 (Pin_2)
- net MICWS: now reaches U1.5 (IO5)
- net MICWS: now also MICCLK1.3 (Pin_3)
- net 6: now reaches U1.6 (IO6)
- net 6: now also J8.1 (Pin_1)
- net 7: now reaches U1.7 (IO7)
- net 7: now also J8.2 (Pin_2)
- net 15: now reaches U1.8 (IO15)
- net 15: now also J3.1 (Pin_1)
- net 16: now reaches U1.9 (IO16)
- net 16: now also J3.2 (Pin_2)
- new net: Q1.1, Q2.2, R10.1
- new net: Q1.2, Q2.1, R11.2
- new net: Q2.3, R9.1
- new net: C5.1, R3.2
- new net: Q1.3, R8.1
- new net CTS: J11.2 (Pin_2), R11.1
- new net DTR: J11.1 (Pin_1), R10.2
- no-connect marks 0 -> 11
Other:
- note added: "Button"
- note added: "DEBUG PRINT"
- note added: "ESP32 MCU"
- note added: "LCD DISPLAY"
- note added: "MIC"
- note added: "Pulldown"
- note added: "SPEAKER"
- moved on the sheet: U1
